File: air-quality-ble-sensor.kicad_sch (KiCad schematic)
At the start: 10 parts, among them J1 SS-52400-002, J2 B2B-PH-SM4-TB, U1 MCP73871

Commit message: continue...
Parts:
- added F1: 0ZCH0110AF2E, FUSC3226X100N, symbol 0ZCH0110AF2E:0ZCH0110AF2E
- added LED1: LTST-C170KRKT, LEDC2012X120N, symbol LTST-C170KRKT:LTST-C170KRKT
- added LED2: LTST-C170GKT, LEDC2012X120N, symbol LTST-C170GKT:LTST-C170GKT
- added LED3: LTST-C170TBKT, LEDC2012X120N, symbol LTST-C170TBKT:LTST-C170TBKT
- added R7, R8, R9: 470R, symbol Device:R
Connections:
- net GND: now also J1.A1 (GNDA1), J1.A12 (GNDA2), J1.B1 (GNDB1), J1.B12 (GNDB2), J1.G1 (GND/SHIELD), J1.G2 (GND/SHIELD), J1.G3 (GND/SHIELD), J1.G4 (GND/SHIELD), J1.S1 (GND/SHIELD), J1.S2 (GND/SHIELD), J1.S3 (GND/SHIELD), J1.S4 (GND/SHIELD), R3.2, R4.2
- net at U1.6 (~{PG}): now also R9.1
- net at U1.7 (STAT2): now also R7.1
- net at U1.8 (STAT1/~{LBO}): now also R8.1
- net at J1.B4 (VBUSB1): now also F1.1
- new net: LED1.1 (K), R7.2
- new net: LED3.1 (K), R9.2
- new net: LED2.1 (K), R8.2
